Commit message: Motion in Gazebo

File: description/robot.urdf.xacro (robot description, xacro)
@@ -1,4 +1,5 @@
 <?xml version="1.0"?>
 <robot xmlns:xacro="http://www.ros.org/wiki/xacro"  name="robot">
-<xacro:include filename="robot_core.xacro" />
+    <xacro:include filename="robot_core.xacro" />
+    <xacro:include filename="gazebo_control.xacro" />
 </robot>

File: description/robot_core.xacro (robot description, xacro)
@@ -41,4 +41,7 @@
         </xacro:inertial_box>
     </link>
+    <gazebo reference="chassis">
+        <material>Gazebo/Orange</material>
+    </gazebo>
     <!-- LEFT WHEEL LINK -->
     <joint name="left_wheel_joint" type="continuous">
@@ -64,4 +67,7 @@
         </xacro:inertial_cylinder>
     </link>
+    <gazebo reference="left_wheel">
+        <material>Gazebo/Blue</material>
+    </gazebo>
     <!-- RIGHT WHEEL LINK -->
     <joint name="right_wheel_joint" type="continuous">
@@ -87,4 +93,7 @@
         </xacro:inertial_cylinder>
     </link>
+    <gazebo reference="right_wheel">
+        <material>Gazebo/Blue</material>
+    </gazebo>
    <!-- FRONT SUPPORT WHEEL -->
 <joint name="front_support_wheel_joint" type="fixed">
@@ -97,5 +106,5 @@
     <visual>
         <geometry>
-            <cylinder radius="0.04" length="0.03"/>
+            <cylinder radius="0.04" length="0.04"/>
         </geometry>
         <material name="blue"/>
@@ -103,11 +112,16 @@
     <collision>
         <geometry>
-            <cylinder radius="0.04" length="0.03"/>
+            <cylinder radius="0.04" length="0.04"/>
         </geometry>
     </collision>
-    <xacro:inertial_cylinder mass="0.05" length="0.03" radius="0.04">
+    <xacro:inertial_cylinder mass="0.05" length="0.04" radius="0.04">
         <origin xyz="0 0 0" rpy="0 0 0"/>
     </xacro:inertial_cylinder>
 </link>
+    <gazebo reference="front_support_wheel">
+        <material>Gazebo/Blue</material>
+        <mu1 value="0.001"/>
+        <mu2 value="0.001"/>
+    </gazebo>
 <!-- REAR SUPPORT WHEEL -->
 <joint name="rear_support_wheel_joint" type="fixed">
@@ -120,5 +134,5 @@
     <visual>
         <geometry>
-            <cylinder radius="0.04" length="0.03"/>
+            <cylinder radius="0.04" length="0.04"/>
         </geometry>
         <material name="blue"/>
@@ -126,10 +140,15 @@
     <collision>
         <geometry>
-            <cylinder radius="0.04" length="0.03"/>
+            <cylinder radius="0.04" length="0.04"/>
         </geometry>
     </collision>
-    <xacro:inertial_cylinder mass="0.05" length="0.03" radius="0.04">
+    <xacro:inertial_cylinder mass="0.05" length="0.04" radius="0.04">
         <origin xyz="0 0 0" rpy="0 0 0"/>
     </xacro:inertial_cylinder>
 </link>
+    <gazebo reference="rear_support_wheel">
+        <material>Gazebo/Blue</material>
+        <mu1 value="0.001"/>
+        <mu2 value="0.001"/>
+    </gazebo>
 </robot>
